File: hardware/kicad/cropdroid-reservoir.kicad_pcb (KiCad board)
At the start: 2 copper layers, 170.4 x 73.7 mm, 23 parts, among them CON1 SJ1-3523N, CON2 SJ1-3523N, CON3 SJ1-3523N, CON4 SJ1-3523N, CON5 SJ1-3523N, CON6 SJ1-3523N, CON7 SJ1-3523N, J1 OSTTC020162, J2 640456-3, J3 OSTTC020162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

Commit message: refactor kicad folder to hardware
Parts:
- added G***: LOGO, cropdroid_logo:cropdroid_logo, F.Cu at (214.6, 83.8)
- moved CON2 0.25 mm to (97.8, 120.4)
