File: hardware/kicad/cropdroid-reservoir.sch (KiCad schematic (older format))
At the start: 23 parts, among them CON1 SJ1-3523N, CON2 SJ1-3523N, CON3 SJ1-3523N, CON4 SJ1-3523N, CON5 SJ1-3523N, CON6 SJ1-3523N, CON7 SJ1-3523N, J1 OSTTC020162, J2 640456-3, J3 OSTTC020162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

Commit message: complete prototype v0.1a
Other:
- note added: "Analog 0"
- note added: "Analog 1"
- note added: "Channel 0"
- note added: "Channel 1"
- note added: "Channel 2"
- note added: "Channel 3"
- note added: "Channel 4"
- note added: "Channel 5"
- note added: "Channel 6"
- note added: "DHT22"
- note added: "OneWire"
Changed lines of the file:
@@
 Wire Wire Line
 	6550 1450 6550 1750
+Text Notes 2300 3100 0    50   ~ 0
+Channel 1
+Text Notes 3350 3050 0    50   ~ 0
+Channel 2
+Text Notes 4400 3050 0    50   ~ 0
+Channel 3
+Text Notes 9500 700  0    50   ~ 0
+Channel 0
+Text Notes 6350 700  0    50   ~ 0
+Channel 4
+Text Notes 7400 700  0    50   ~ 0
+Channel 5
+Text Notes 8450 700  0    50   ~ 0
+Channel 6
+Text Notes 3150 6300 0    50   ~ 0
+Analog 0
+Text Notes 7050 6350 0    50   ~ 0
+Analog 1
+Text Notes 1250 4250 0    50   ~ 0
+OneWire
+Text Notes 1850 4750 0    50   ~ 0
+DHT22
+Text Notes 8650 3450 0    50   ~ 0
+Channel 0
 $EndSCHEMATC
