File: hardware/kicad/cropdroid-reservoir-120v/cropdroid-reservoir.kicad_pcb (KiCad board)
At the start: 2 copper layers, 170.4 x 73.7 mm, 24 parts, among them CON1 SJ1-3523N, CON2 SJ1-3523N, CON3 SJ1-3523N, CON4 SJ1-3523N, CON5 SJ1-3523N, CON6 SJ1-3523N, CON7 SJ1-3523N, J1 OSTTC020162, J2 640456-3, J3 OSTTC020162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

Commit message: add cropdroid-reservoir-120v design
Parts:
- removed the G*** at (214.6, 83.8)
- removed J2: 640456-3, digikey-footprints:PinHeader_1x3_P2.54_Drill1.1mm
- added D4: LED, libraries:CAPPRD350W60D800H2000, F.Cu at (130.0, 111.0)
- added D5: 1N4001, Diode_THT:D_DO-41_SOD81_P10.16mm_Horizontal, F.Cu at (172.2, 105.7)
- added D6: LED, libraries:CAPPRD350W60D800H2000, F.Cu at (180.3, 111.0)
- added G***: LOGO, libraries:cropdroid_logo, F.Cu at (38.1, 27.9)
- added J12: 703W-00_52, 703W-00_54:52, F.Cu at (271.0, 42.4)
- added J7: TB005-762-02BE, TB005-762-02BE:CUI_TB005-762-02BE, F.Cu at (166.6, 46.7)
- added J8: 3-213598-2, 3-213598-2:TE_3-213598-2, F.Cu at (187.2, 48.3)
- added J9: TB005-762-02BE, TB005-762-02BE:CUI_TB005-762-02BE, F.Cu at (216.9, 47.0)
- added PS1: PSK-6B-S5, PSK-6B-S5:CONV_PSK-6B-S5, F.Cu at (256.3, 86.6)
- added R1: 4.7k, Resistor_THT:R_Axial_DIN0207_L6.3mm_D2.5mm_P10.16mm_Horizontal, F.Cu at (31.8, 195.3)
- added R2: 10k, Resistor_THT:R_Axial_DIN0207_L6.3mm_D2.5mm_P10.16mm_Horizontal, F.Cu at (76.7, 156.7)
- added R5: R, Resistor_THT:R_Axial_DIN0207_L6.3mm_D2.5mm_P10.16mm_Horizontal, F.Cu at (180.8, 118.4)
- added Screw: Drill, drill-hole:Drill_Hole, F.Cu at (247.7, 63.5)
- added Screw: Drill, drill-hole:Drill_Hole, F.Cu at (31.8, 127.0)
- added Screw: Drill, drill-hole:Drill_Hole, F.Cu at (279.4, 190.5)
- added Screw: Drill, drill-hole:Drill_Hole, F.Cu at (63.5, 25.4)
- added U1: IRM-30-12, IRM-30-12:IRM-30-12, F.Cu at (281.9, 119.4)
- D2: value 1N4001 -> LED; footprint Diode_THT:D_DO-41_SOD81_P10.16mm_Horizontal -> libraries:CAPPRD350W60D800H2000
- J1: value OSTTC020162 -> 640456-3; footprint digikey-footprints:Term_Block_1x2_P5mm -> digikey-footprints:PinHeader_1x3_P2.54_Drill1.1mm
- J3: value OSTTC020162 -> 3-213598-2; footprint digikey-footprints:Term_Block_1x2_P5mm -> 3-213598-2:TE_3-213598-2
- J4: value OSTTC020162 -> TB005-762-02BE; footprint digikey-footprints:Term_Block_1x2_P5mm -> TB005-762-02BE:CUI_TB005-762-02BE
- J6: value PJ-102A -> 3-213598-2; footprint digikey-footprints:Barrel_Jack_5.5mmODx2.1mmID_PJ-102A -> 3-213598-2:TE_3-213598-2
- R3: value 10k -> R
- R4: value 4.7k -> R
- moved CON1 169.6 mm to (42.5, 185.9)
- moved R3 156.5 mm to (79.5, 118.4), turned to 0 degrees
- moved CON4 118.4 mm to (83.6, 185.9)
- moved J1 108.5 mm to (70.4, 164.6), turned to 90 degrees
- moved J6 102.8 mm to (136.9, 47.5), turned to 0 degrees
- moved Q1 100.9 mm to (31.8, 165.9), turned to 90 degrees
- moved J5 91.9 mm to (16.8, 172.7)
- moved CON7 87.8 mm to (166.4, 185.9)
- moved D2 78.8 mm to (79.8, 111.0), turned to 180 degrees
- moved CON2 72.3 mm to (67.3, 185.9)
- moved RLY1 71.8 mm to (169.4, 162.8), turned to 270 degrees
- moved J4 68.4 mm to (115.8, 46.5)
- moved D3 68.2 mm to (121.9, 105.7)
- moved CON3 67.9 mm to (109.2, 185.9)
- moved CON5 67.7 mm to (125.5, 185.9)
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Connections:
- D2 pad 1: +12V -> Net-(D2-Pad1)
- D2 pad 2: Net-(D2-Pad2) -> +12V
- J1 pad 1: Net-(J1-Pad1) -> Net-(CON1-Pad3)
- J3 pad 1: Net-(J3-Pad1) -> Net-(J12-Pad3)
- J4 pad 1: Net-(J4-Pad1) -> Net-(J12-Pad1)
- J4 pad 2: Net-(J4-Pad2) -> Net-(J3-Pad2)
- J5 pad 1: Net-(CON2-Pad3) -> Net-(CON1-Pad3)
- J5 pad 19: Net-(CON2-Pad2) -> Net-(CON1-Pad2)
- J5 pad 21: Net-(CON1-Pad2) -> Net-(CON2-Pad2)
- J5 pad 22: Net-(J2-Pad2) -> Net-(J1-Pad2)
- J6 pad 1: +12V -> Net-(J12-Pad3)
- J6 pad 2: GND -> Net-(J6-Pad2)
- J6 pad 3: Net-(J6-Pad3) -> Net-(J12-Pad2)
- K1 pad 3: Net-(J1-Pad2) -> Net-(J12-Pad1)
- K1 pad 4: Net-(J1-Pad1) -> Net-(J3-Pad2)
- K2 pad 1: Net-(D2-Pad2) -> Net-(D3-Pad2)
- K2 pad 3: Net-(J3-Pad2) -> Net-(J12-Pad1)
- K2 pad 4: Net-(J3-Pad1) -> Net-(J6-Pad2)
- K3 pad 1: Net-(D3-Pad2) -> Net-(D5-Pad2)
- K3 pad 3: Net-(J4-Pad2) -> Net-(J12-Pad1)
- K3 pad 4: Net-(J4-Pad1) -> Net-(J8-Pad2)
- Q1 pad 13: Net-(D3-Pad2) -> Net-(D5-Pad2)
- Q1 pad 14: Net-(D2-Pad2) -> Net-(D3-Pad2)
- R3 pad 1: Net-(J2-Pad2) -> Net-(D2-Pad1)
- R3 pad 2: Net-(CON2-Pad3) -> GND
- R4 pad 1: Net-(CON2-Pad2) -> Net-(D4-Pad1)
- R4 pad 2: Net-(CON2-Pad3) -> GND
Routing:
- net Net-(J12-Pad1): track 0.00 -> 576.7 mm
- net Net-(J12-Pad2): track 0.00 -> 514.3 mm
- net Net-(CON1-Pad3): track 0.00 -> 504.9 mm
- net GND: track 5.62 -> 325.0 mm
- net Net-(J12-Pad3): track 0.00 -> 317.1 mm
- net +12V: track 301.0 -> 565.6 mm
- net Net-(CON2-Pad3): track 233.1 -> 0.00 mm
- net Net-(J2-Pad2): track 225.1 -> 0.00 mm
- net Net-(D5-Pad2): track 0.00 -> 171.4 mm
- net Net-(CON1-Pad2): track 172.9 -> 59.3 mm
- net Net-(D2-Pad2): track 82.3 -> 0.00 mm
- net Net-(CON4-Pad2): track 149.6 -> 76.4 mm
- net Net-(J6-Pad2): track 0.00 -> 50.3 mm
- net Net-(J8-Pad2): track 0.00 -> 49.3 mm
- net Net-(CON7-Pad1): track 72.7 -> 26.2 mm
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Other:
- board size 170.4 x 73.7 mm -> 273.9 x 190.2 mm
- net class MainsAC added: clearance 3.048, trace_width 3.81, via_dia 2.032, via_drill 0.381
- board text added: "+12v DC"
- board text added: "+5V DC"
- board text added: "120v AC"
- board text added: "Channel0"
- board text added: "Channel1"
- board text added: "Channel2"
- board text added: "Channel3"
- board text added: "Channel4"
- board text added: "Channel5"
- board text added: "Channel6"
- board text added: "CropDroid Reservoir Controller CopyRight (c) Automate The Things, LLC Prototype v0.3a"
- board text added: "Ground"
- board text added: "Line"
- board text added: "Neutral"
- board text removed: "Channel 1"
- board text removed: "Channel 2"
- board text removed: "Channel 3"
- board text removed: "Channel 4"
- board text removed: "Channel 5"
- board text removed: "Channel 6"
- board text removed: "CropDroid Reservoir Controller Copyright (c) Automate The Things, LLC Prototype v0.1a"
- board text removed: "Drain Channel 0"
