File: hardware/kicad/cropdroid-reservoir-120v/cropdroid-reservoir.kicad_pcb (KiCad board)
At the start: 2 copper layers, 273.9 x 190.2 mm, 39 parts, among them CON1 SJ1-3523N, CON2 SJ1-3523N, CON3 SJ1-3523N, CON4 SJ1-3523N, CON5 SJ1-3523N, CON6 SJ1-3523N, CON7 SJ1-3523N, J1 640456-3, J12 703W-00_52, J3 3-213598-2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

Commit message: final kicad v0.2a
Parts:
- removed the CON2 at (67.3, 185.9)
- removed J12: 703W-00_52, 703W-00_54:52
- removed the J3 at (86.6, 47.5)
- removed the J4 at (115.8, 46.5)
- removed J7, J9: TB005-762-02BE, TB005-762-02BE:CUI_TB005-762-02BE
- removed J8: 3-213598-2, 3-213598-2:TE_3-213598-2
- added CON1: SJ1-3523N, digikey-footprints:Headphone_Jack_3.5mm_SJ1-3523N, F.Cu at (126.1, 207.9)
- added CON7: SJ1-3523N, digikey-footprints:Headphone_Jack_3.5mm_SJ1-3523N, F.Cu at (223.3, 207.9)
- added J2: 3-213598-2, 3-213598-2:TE_3-213598-2, F.Cu at (142.9, 62.2)
- added J5: 3-213598-2, 3-213598-2:TE_3-213598-2, F.Cu at (243.5, 62.2)
- J1: value 640456-3 -> 703W-00_52; footprint digikey-footprints:PinHeader_1x3_P2.54_Drill1.1mm -> 703W-00_52:QUALTEK_703W-00_52
- moved J1 269.2 mm to (326.6, 82.0)
- moved CON4 109.3 mm to (190.6, 207.9)
- moved CON8 82.6 mm to (246.0, 207.9)
- moved RLY1 82.6 mm to (249.0, 184.8)
- moved CON6 68.8 mm to (206.9, 207.9)
- moved R2 65.7 mm to (131.2, 193.5), turned to 180 degrees
- moved R1 64.9 mm to (92.8, 217.4)
- moved CON2 64.8 mm to (103.4, 208.0)
- moved G*** 62.3 mm to (89.5, 63.1)
- moved R3 59.8 mm to (135.1, 140.4)
- moved D1 59.8 mm to (126.7, 127.4)
- moved J3 59.8 mm to (72.3, 194.8)
- moved Q1 59.8 mm to (87.3, 187.9)
- moved R4 59.8 mm to (185.9, 140.4)
- moved R5 59.8 mm to (236.4, 140.4)
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- renumbered CON1 to CON2, CON7 to CON8, J5 to J3, J6 to J4
Connections:
- CON3 pad 1: +12V -> GND
- CON4 pad 1: GND -> +12V
- CON5 pad 1: +12V -> GND
- J1 pad 1: Net-(CON1-Pad3) -> Net-(J1-Pad1)
- J1 pad 3: GND -> Net-(J1-Pad3)
- J3 pad 20: Net-(CON4-Pad2) -> Net-(CON5-Pad2)
- J3 pad 21: Net-(CON2-Pad2) (its old number) -> Net-(CON3-Pad2)
- J3 pad 22: Net-(J1-Pad2) -> Net-(CON1-Pad2)
- J4 pad 1: Net-(J12-Pad3) -> Net-(J1-Pad3)
- J4 pad 3: Net-(J12-Pad2) -> Net-(J1-Pad2)
- K1 pad 3: Net-(J12-Pad1) -> Net-(J1-Pad1)
- K2 pad 3: Net-(J12-Pad1) -> Net-(J1-Pad1)
- K3 pad 3: Net-(J12-Pad1) -> Net-(J1-Pad1)
- PS1 pad 1: Net-(J12-Pad2) -> Net-(J1-Pad3)
- PS1 pad 2: Net-(J12-Pad1) -> Net-(J1-Pad1)
- Q1 pad 10: Net-(CON6-Pad2) -> Net-(CON7-Pad2)
- Q1 pad 11: Net-(CON5-Pad2) -> Net-(CON6-Pad2)
- Q1 pad 12: Net-(CON3-Pad2) -> Net-(CON4-Pad2)
- R2 pad 1: Net-(J1-Pad2) -> Net-(CON1-Pad2)
- U1 pad 1: Net-(J12-Pad1) -> Net-(J1-Pad1)
- U1 pad 2: Net-(J12-Pad2) -> Net-(J1-Pad3)
Routing:
- net Net-(J12-Pad1): track 576.7 -> 0.00 mm
- net Net-(J12-Pad2): track 514.3 -> 0.00 mm
- net Net-(J1-Pad1): track 0.00 -> 432.1 mm
- net Net-(J1-Pad3): track 0.00 -> 392.5 mm
- net Net-(J12-Pad3): track 317.1 -> 0.00 mm
- net GND: track 325.0 -> 41.2 mm
- net Net-(J1-Pad2): track 66.9 -> 311.6 mm
- net Net-(CON7-Pad2): track 0.00 -> 142.5 mm
- net Net-(CON1-Pad3): track 504.9 -> 375.7 mm
- net Net-(CON1-Pad2): track 0.00 -> 75.0 mm
- net Net-(CON2-Pad2) (its old number): track 61.7 -> 0.00 mm
- net Net-(CON4-Pad2): track 76.4 -> 116.3 mm
- net +12V: track 565.6 -> 530.5 mm
- net Net-(Q1-Pad16): track 145.0 -> 169.3 mm
- net Net-(CON6-Pad2): track 117.3 -> 130.2 mm
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Other:
- board size 273.9 x 190.2 mm -> 273.9 x 168.8 mm
- net class MainsAC: trace_width 3.81 -> 5.08
- board text added: "DHT22 / AM2303"
- board text added: "Earth"
- board text removed: "120v AC"
- board text removed: "Ground"

Commit message: final v0.3a iterations
Other:
- rule pad_to_mask_clearance: 0.051 -> 0.0508
Changed lines of the file:
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@@
   )
   (setup
-    (last_trace_width 2.794)
+    (last_trace_width 0.254)
     (user_trace_width 0.762)
     (user_trace_width 2.794)
@@
     (pad_size 4.2 4.2)
     (pad_drill 3.2)
-    (pad_to_mask_clearance 0.051)
-    (solder_mask_min_width 0.25)
+    (pad_to_mask_clearance 0.0508)
     (aux_axis_origin 0 0)
     (grid_origin 68.9102 218.3638)
