File: hardware/kicad/cropdroid-reservoir-120v/cropdroid-reservoir.sch (KiCad schematic (older format))
At the start: 34 parts, among them CON1 SJ1-3523N, CON2 SJ1-3523N, CON3 SJ1-3523N, CON4 SJ1-3523N, CON5 SJ1-3523N, CON6 SJ1-3523N, CON7 SJ1-3523N, J1 640456-3, J12 703W-00_52, J3 3-213598-2, J4 TB005-762-02BE, J5 SAMTEC-MTSW-118-10-X-D-640, J6 3-213598-2, J7 TB005-762-02BE, J8 3-213598-2, J9 TB005-762-02BE, K1 T9AS1D12-15, K2 T9AS1D12-15, K3 T9AS1D12-15, Q1 ULN2003AN, U1 IRM-30-12

Commit message: final kicad v0.2a
Parts:
- removed J1: 640456-3, digikey-footprints:PinHeader_1x3_P2.54_Drill1.1mm, symbol dk_Rectangular-Connectors-Headers-Male-Pins:640456-3
- removed J12: 703W-00_52, 703W-00_54:52, symbol 703W-00_52:703W-00_52
- removed J4, J7, J9: TB005-762-02BE, TB005-762-02BE:CUI_TB005-762-02BE, symbol TB005-762-02BE:TB005-762-02BE
- added CON1: SJ1-3523N, digikey-footprints:Headphone_Jack_3.5mm_SJ1-3523N, symbol dk_Barrel-Audio-Connectors:SJ1-3523N
- added J1: 703W-00_52, QUALTEK_703W-00_52, symbol 703W-00_52:703W-00_52
- renumbered CON1 to CON2, CON2 to CON3, CON3 to CON4, CON4 to CON5, CON5 to CON6, CON6 to CON7, CON7 to CON8, J3 to J2, J5 to J3, J6 to J4, J8 to J5
Connections:
- net GND: now also CON1.1 (S)
- net at CON2.3 (R), J3.1, PS1.3 (+VOUT)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: now also CON1.3 (R)
- net at J3.22, R2.1: now also CON1.2 (T)
- net at K1.3 (C), K2.3 (C), K3.3 (C)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: now also J1.1 (L)
- net at J2.3, J4.3, J5.3: now also J1.2 (E)
- net at J2.1, J4.1, J5.1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: now also J1.3 (N)
Other:
- moved on the sheet: R2
