File: hardware/kicad/cropdroid-reservoir-v0.5a/cropdroid-reservoir.kicad_pcb (KiCad board)
At the start: 2 copper layers, 316.2 x 168.8 mm, 42 parts, among them CON1 SJ1-3523N, CON2 SJ1-3523N, CON3 SJ1-3523N, CON4 SJ1-3523N, CON5 SJ1-3523N, CON6 SJ1-3523N, CON7 SJ1-3523N, CON8 SJ1-3523N, J1 703W-00_52, J2 3-213598-2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

Commit message: v0.5a final
Parts:
- moved Screw 27.1 mm to (64.6, 118.0)
- moved G*** 6.86 mm to (72.2, 51.7)
- moved Screw 4.85 mm to (95.1, 62.7)
Routing:
- net Net-(J1-Pad2): track 267.7 -> 249.2 mm
- net Net-(J1-Pad3): track 410.8 -> 429.1 mm
Other:
- board size 316.2 x 168.8 mm -> 316.2 x 175.7 mm

Commit message: v0.5a final
Parts:
- moved Screw 10.5 mm to (95.2, 52.1)
- moved Screw 5.91 mm to (318.1, 98.0)
- moved G*** 3.67 mm to (71.3, 48.1)
Other:
- board size 316.2 x 175.7 mm -> 316.2 x 178.2 mm
Changed lines of the file:
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@@
   )
   (setup
-    (last_trace_width 5.08)
+    (last_trace_width 0.254)
     (user_trace_width 0.762)
     (user_trace_width 2.794)
@@
   )
   (module drill-hole:Drill_Hole (layer F.Cu)
-    (at 95.0722 62.6618)
+    (at 95.1992 52.1208)
     (fp_text reference Screw (at -0.254 3.556) (layer F.SilkS)
       (effects (font (size 1 1) (thickness 0.15)))
@@
   )
   (module drill-hole:Drill_Hole (layer F.Cu)
-    (at 317.1952 92.1258)
+    (at 318.0842 97.9678)
     (fp_text reference Screw (at -0.127 3.302) (layer F.SilkS)
       (effects (font (size 1 1) (thickness 0.15)))
@@
   )
   (module libraries:cropdroid_logo (layer F.Cu)
-    (at 72.2376 51.6509)
+    (at 71.3486 48.0949)
     (fp_text reference G*** (at 0 0) (layer F.SilkS) hide
       (effects (font (size 1.524 1.524) (thickness 0.3)))
@@
     (effects (font (size 1 1) (thickness 0.15)))
   )
-  (gr_line (start 51.3715 38.1) (end 51.6382 213.7918) (layer Edge.Cuts) (width 0.05))
+  (gr_line (start 51.3715 35.56) (end 51.6382 213.7918) (layer Edge.Cuts) (width 0.05))
   (gr_text "+12v DC" (at 289.1282 185.5978) (layer F.SilkS)
     (effects (font (size 1 1) (thickness 0.15)))
@@
     (effects (font (size 1 1) (thickness 0.15)))
   )
-  (gr_text "CropDroid Reservoir Controller\nCopyRight (c) Automate The Things, LLC\nPrototype v0.4a" (at 53.1876 42.7609) (layer F.SilkS)
+  (gr_text "CropDroid Reservoir Controller\nCopyRight (c) Automate The Things, LLC\nPrototype v0.4a" (at 52.2986 39.2049) (layer F.SilkS)
     (effects (font (size 1 1) (thickness 0.15)) (justify left))
   )
   (gr_line (start 367.6015 213.7918) (end 51.6382 213.7918) (layer Edge.Cuts) (width 0.05))
-  (gr_line (start 367.6015 38.1) (end 367.6015 213.7918) (layer Edge.Cuts) (width 0.05))
-  (gr_line (start 51.3715 38.1) (end 367.6015 38.1) (layer Edge.Cuts) (width 0.05))
+  (gr_line (start 367.6015 35.56) (end 367.6015 213.7918) (layer Edge.Cuts) (width 0.05))
+  (gr_line (start 51.3715 35.56) (end 367.6015 35.56) (layer Edge.Cuts) (width 0.05))
   (segment (start 113.8644 189.0052) (end 113.8936 188.976) (width 0.254) (layer B.Cu) (net 1) (status 30))
   (segment (start 113.8644 203.3778) (end 113.8644 189.0052) (width 0.254) (layer B.Cu) (net 1) (status 30))

Commit message: remove xml bom
Other:
- board size 316.2 x 178.2 mm -> 316.2 x 178.4 mm
Changed lines of the file:
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@@
     (effects (font (size 1 1) (thickness 0.15)))
   )
-  (gr_line (start 51.3715 35.56) (end 51.6382 213.7918) (layer Edge.Cuts) (width 0.05))
+  (gr_line (start 51.3715 35.433) (end 51.6382 213.7918) (layer Edge.Cuts) (width 0.05))
   (gr_text "+12v DC" (at 289.1282 185.5978) (layer F.SilkS)
     (effects (font (size 1 1) (thickness 0.15)))
@@
   )
   (gr_line (start 367.6015 213.7918) (end 51.6382 213.7918) (layer Edge.Cuts) (width 0.05))
-  (gr_line (start 367.6015 35.56) (end 367.6015 213.7918) (layer Edge.Cuts) (width 0.05))
-  (gr_line (start 51.3715 35.56) (end 367.6015 35.56) (layer Edge.Cuts) (width 0.05))
+  (gr_line (start 367.6015 35.433) (end 367.6015 213.7918) (layer Edge.Cuts) (width 0.05))
+  (gr_line (start 51.3715 35.433) (end 367.6015 35.433) (layer Edge.Cuts) (width 0.05))
   (segment (start 113.8644 189.0052) (end 113.8936 188.976) (width 0.254) (layer B.Cu) (net 1) (status 30))
   (segment (start 113.8644 203.3778) (end 113.8644 189.0052) (width 0.254) (layer B.Cu) (net 1) (status 30))
