File: hardware/kicad/cropdroid-reservoir-v0.6a/cropdroid-reservoir.sch (KiCad schematic (older format))
At the start: 37 parts, among them J1 703W-00_52, J10 PJ-102A, J11 PJ-102A, J12 PJ-102A, J13 PJ-102A, J14 PJ-102A, J2 2172034-1, J3 2172034-1, J4 PJ-102A, J5 3-213598-2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

Commit message: add /sys endpoint
Other:
- note added: "Channel 7"
Changed lines of the file:
@@
 Channel 0
 Text Notes 7250 800  0    50   ~ 0
-Channel 4
+Channel 5
 Text Notes 8300 800  0    50   ~ 0
-Channel 5
+Channel 6
 Text Notes 9250 800  0    50   ~ 0
-Channel 6
+Channel 7
 Text Notes 2900 6450 0    50   ~ 0
 Analog 0
@@
 	6250 2850 6250 2950
 Text Notes 6350 3450 0    50   ~ 0
-Channel 3
+Channel 4
 Wire Wire Line
 	5950 2850 6250 2850
